File: Hardware/KiCad/usb_ethernet_uart_bridge.kicad_sch (KiCad schematic)
At the start: 13 parts, among them U1 XR22801IL32TR-F, Y1 ABM8-25.000MHZ-B2-T3

Commit message: Rename all MDI signals to match kicad diffpair naming scheme
Connections:
- net MDI_RN_P0 renamed MDI_P0_RN
- net MDI_RP_P0 renamed MDI_P0_RP
- net MDI_TN_P0 renamed MDI_P0_TN
- net MDI_TP_P0 renamed MDI_P0_TP
Changed lines of the file:
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@@
 		)
 	)
-	(global_label "MDI_TN_P0"
+	(global_label "MDI_P0_TN"
 		(shape input)
 		(at 27.94 147.32 180)
@@
 		)
 	)
-	(global_label "MDI_RN_P0"
+	(global_label "MDI_P0_RN"
 		(shape input)
 		(at 27.94 160.02 180)
@@
 		)
 	)
-	(global_label "MDI_TP_P0"
+	(global_label "MDI_P0_TP"
 		(shape input)
 		(at 27.94 153.67 180)
@@
 		)
 	)
-	(global_label "MDI_RP_P0"
+	(global_label "MDI_P0_RP"
 		(shape input)
 		(at 27.94 166.37 180)
